File: hardware/integrated/toshiba_hvac_esp32_integrated.kicad_pcb (KiCad board)
At the start: 2 copper layers, 29 x 50.3 mm, 35 parts, among them J1 S05B-PASK-2LFSN, J2 TYPE-C-31-M-12, Q1 S8050, Q2 S8050, SW1 EN, SW2 BOOT, U1 ESP32-WROOM-32E-N8, U2 TXS0108EPW, U3 AMS1117-3.3, U4 CP2102N-A02-GQFN24

Commit message: fix(hw): USB-C mating face pointed into the board
J2's signal pins sat east of its shell posts, so the connector opening
faced the board interior instead of the east edge - the port could not
have been plugged in. Found in JLCPCB's placement preview; invisible in
KiCad's own render because the library ships no 3D model for this part.

Rotated J2 180deg and moved it east so the body is flush with the board
outline. Its pads move from x 62.945 to x 56.315, so the whole USB block
is re-routed: staggered D+/D- via columns west of the pad field, CC1 and
CC2 escaping south to relocated pulldowns, and VBUS looping east under
the connector body to tie both power pads.

build_pcb.py now asserts the orientation so this cannot regress.
DRC 0 errors / 0 unconnected; schematic-PCB parity 0 mismatches.

Also adds jlc_cpl_fix.py: positions.csv now carries a +270deg correction
for U1 (JLCPCB's module model has a different zero-orientation) and a
centroid shift for J1 (footprint anchor is pad 1, JLCPCB wants centre).
Parts:
- moved R7 6.14 mm to (52.2, 70.4), turned to 180 degrees
- moved J2 1.46 mm to (60.4, 64.7), turned to 90 degrees
- moved R6 0.76 mm to (59.2, 71.4), turned to 0 degrees
Routing:
- net USB_DP: track 18.2 -> 12.5 mm
- net USB_DM: track 19.1 -> 14.6 mm
- net VBUS: track 37.1 -> 33.1 mm, vias 5 -> 3
- net CC2: track 9.56 -> 11.0 mm
- net GND: track 4.20 -> 3.54 mm
